Commit message: Working 1 finger jacobian

File: matlab_jaco/3dof.urdf (robot description, URDF)
Before this commit: robot simple_serial_robot, 4 links, 3 joints
Links:
- added link link_eef; visual sphere radius=0.05
- link arm_base: geometry visual box size=0.11 0.15 0.35
- link base_link: geometry visual box size=0.6 0.6 0.01
- link link2: geometry visual box size=0.05 0.05 0.2
Joints:
- added joint joint_eef: type fixed, parent link2, child link_eef, origin xyz=0 0 0.2
- joint joint1: origin xyz=0 0 0.025 -> xyz=0 0 0
- joint joint2: limit lower=-3.14 upper=3.14 effort=1000.0 velocity=0.5 -> lower=-1.57 upper=1.57 effort=1000.0 velocity=0.5; origin xyz=0.0 0 0.05 -> xyz=0 0 0.35
- joint joint3: limit lower=-3.14 upper=3.14 effort=1000.0 velocity=0.5 -> lower=-1.57 upper=1.57 effort=1000.0 velocity=0.5
